File: ECU_Front/ECU_Front/ECU_Front.kicad_sch (KiCad schematic)
At the start: 18 parts, among them J1 Conn_01x04_Pin, U1 step-down (buck), U4 ESP32-DevKitC

Commit message: ECU_Front, definitive edition
Parts:
- removed U1: step-down (buck), StepDown:StepDown_LM2596, symbol Regulator_Switching:TSR_1-2412
- added J3: Conn_01x02_Pin, Connector_PinHeader_2.54mm:PinHeader_1x02_P2.54mm_Vertical, symbol Connector:Conn_01x02_Pin
- added U2: YAAJ_DCDC_StepDown_LM2596, StepDown:StepDown_LM2596, symbol StepDown_LM2596:YAAJ_DCDC_StepDown_LM2596
- J1: footprint Connector:FanPinHeader_1x04_P2.54mm_Vertical -> Connector:NS-Tech_Grove_1x04_P2mm_Vertical
Connections:
- net +12V: now also J3.1 (Pin_1), U2.1 (Vin)
- net +5V: now also U2.4 (Vout)
- net GND: now also J3.2 (Pin_2), U2.2 (GND), U2.3 (GND)
